Commit message: fix:修改了b1_config中的关节角度和初始高度，原本直接复制的a1

File: resources/robots/b1/urdf/b1.urdf (robot description, URDF)
Before this commit: robot b1_description, 36 links, 35 joints
Links:
- link FL_calf: geometry collision mesh filename=/home/myc/isaacgym/legged_gym/resources/robots/b1/meshes/ca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 scale=1 1 1; visual mesh filename=/home/myc/isaacgym/legged_gym/resources/robots/b1/meshes/ca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 scale=1 1 1
- link FL_hip: geometry collision mesh filename=/home/myc/isaacgym/legged_gym/resources/robots/b1/meshes/hi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 scale=1 1 1; visual mesh filename=/home/myc/isaacgym/legged_gym/resources/robots/b1/meshes/hi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 scale=1 1 1
- link FL_thigh: geometry collision mesh filename=/home/myc/isaacgym/legged_gym/resources/robots/b1/meshes/th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 scale=1 1 1; visual mesh filename=/home/myc/isaacgym/legged_gym/resources/robots/b1/meshes/th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 scale=1 1 1
- link FR_calf: geometry collision mesh filename=/home/myc/isaacgym/legged_gym/resources/robots/b1/meshes/ca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 scale=1 1 1; visual mesh filename=/home/myc/isaacgym/legged_gym/resources/robots/b1/meshes/ca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 scale=1 1 1
- link FR_hip: geometry collision mesh filename=/home/myc/isaacgym/legged_gym/resources/robots/b1/meshes/hi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 scale=1 1 1; visual mesh filename=/home/myc/isaacgym/legged_gym/resources/robots/b1/meshes/hi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 scale=1 1 1
- link FR_thigh: geometry collision mesh filename=/home/myc/isaacgym/legged_gym/resources/robots/b1/meshes/th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 scale=1 1 1; visual mesh filename=/home/myc/isaacgym/legged_gym/resources/robots/b1/meshes/th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 scale=1 1 1
- link RL_calf: geometry collision mesh filename=/home/myc/isaacgym/legged_gym/resources/robots/b1/meshes/ca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 scale=1 1 1; visual mesh filename=/home/myc/isaacgym/legged_gym/resources/robots/b1/meshes/ca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 scale=1 1 1
- link RL_hip: geometry collision mesh filename=/home/myc/isaacgym/legged_gym/resources/robots/b1/meshes/hi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 scale=1 1 1; visual mesh filename=/home/myc/isaacgym/legged_gym/resources/robots/b1/meshes/hi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 scale=1 1 1
- link RL_thigh: geometry collision mesh filename=/home/myc/isaacgym/legged_gym/resources/robots/b1/meshes/th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 scale=1 1 1; visual mesh filename=/home/myc/isaacgym/legged_gym/resources/robots/b1/meshes/th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 scale=1 1 1
- link RR_calf: geometry collision mesh filename=/home/myc/isaacgym/legged_gym/resources/robots/b1/meshes/ca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 scale=1 1 1; visual mesh filename=/home/myc/isaacgym/legged_gym/resources/robots/b1/meshes/ca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 scale=1 1 1
- link RR_hip: geometry collision mesh filename=/home/myc/isaacgym/legged_gym/resources/robots/b1/meshes/hi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 scale=1 1 1; visual mesh filename=/home/myc/isaacgym/legged_gym/resources/robots/b1/meshes/hi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 scale=1 1 1
- link RR_thigh: geometry collision mesh filename=/home/myc/isaacgym/legged_gym/resources/robots/b1/meshes/th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 scale=1 1 1; visual mesh filename=/home/myc/isaacgym/legged_gym/resources/robots/b1/meshes/th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 scale=1 1 1
- link trunk: geometry collision mesh filename=/home/myc/isaacgym/legged_gym/resources/robots/b1/meshes/tr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 scale=1 1 1; visual mesh filename=/home/myc/isaacgym/legged_gym/resources/robots/b1/meshes/tr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 scale=1 1 1

File: resources/robots/b1/urdf/b1_stl.urdf (robot description, URDF)
Before this commit: robot b1_description, 36 links, 35 joints
Links:
- link FL_calf: geometry collision mesh filename=../meshes/calfb.stl scale=1 1 1; visual mesh filename=../meshes/calfb.stl scale=1 1 1
- link FL_hip: geometry collision mesh filename=../meshes/hipb.stl scale=1 1 1; visual mesh filename=../meshes/hipb.stl scale=1 1 1
- link FL_thigh: geometry collision mesh filename=../meshes/thighb.stl scale=1 1 1; visual mesh filename=../meshes/thighb.stl scale=1 1 1
- link FR_calf: geometry collision mesh filename=../meshes/calfb.stl scale=1 1 1; visual mesh filename=../meshes/calfb.stl scale=1 1 1
- link FR_hip: geometry collision mesh filename=../meshes/hipb.stl scale=1 1 1; visual mesh filename=../meshes/hipb.stl scale=1 1 1
- link FR_thigh: geometry collision mesh filename=../meshes/thigh_mirrorb.stl scale=1 1 1; visual mesh filename=../meshes/thigh_mirrorb.stl scale=1 1 1
- link RL_calf: geometry collision mesh filename=../meshes/calfb.stl scale=1 1 1; visual mesh filename=../meshes/calfb.stl scale=1 1 1
- link RL_hip: geometry collision mesh filename=../meshes/hipb.stl scale=1 1 1; visual mesh filename=../meshes/hipb.stl scale=1 1 1
- link RL_thigh: geometry collision mesh filename=../meshes/thighb.stl scale=1 1 1; visual mesh filename=../meshes/thighb.stl scale=1 1 1
- link RR_calf: geometry collision mesh filename=../meshes/calfb.stl scale=1 1 1; visual mesh filename=../meshes/calfb.stl scale=1 1 1
- link RR_hip: geometry collision mesh filename=../meshes/hipb.stl scale=1 1 1; visual mesh filename=../meshes/hipb.stl scale=1 1 1
- link RR_thigh: geometry collision mesh filename=../meshes/thigh_mirrorb.stl scale=1 1 1; visual mesh filename=../meshes/thigh_mirrorb.stl scale=1 1 1
- link trunk: geometry collision mesh filename=../meshes/trunkb.stl scale=1 1 1; visual mesh filename=../meshes/trunkb.stl scale=1 1 1

Commit message: 修改urdf和mujoco使用的xml,修改了mujoco运行脚本

File: resources/robots/b1/urdf/b1.urdf (robot description, URDF)
Before this commit: robot b1_description, 36 links, 35 joints
Links:
- removed link FL_calf_rotor
- removed link FL_hip_rotor
- removed link FL_thigh_rotor
- removed link FR_calf_rotor
- removed link FR_hip_rotor
- removed link FR_thigh_rotor
- removed link RL_calf_rotor
- removed link RL_hip_rotor
- removed link RL_thigh_rotor
- removed link RR_calf_rotor
- removed link RR_hip_rotor
- removed link RR_thigh_rotor
- removed link head_camera_1_link
- removed link head_camera_2_link
- removed link left_side_camera_link
- removed link right_side_camera_link
- removed link tail_camera_link
- link FL_calf: mass 1.05 -> 0.207; geometry collision box size=0.35 0.04 0.03; visual mesh filename=../meshes/calf.stl scale=1 1 1
- link FL_foot: mass 0.05 -> 0.06
- link FL_hip: mass 2.15 -> 1.993; geometry collision cylinder length=0.04 radius=0.09; visual mesh filename=../meshes/hip.stl scale=1 1 1
- link FL_thigh: mass 4.3 -> 0.639; geometry collision box size=0.35 0.05 0.08; visual mesh filename=../meshes/thigh.stl scale=1 1 1
- link FR_calf: mass 1.05 -> 0.207; geometry collision box size=0.35 0.04 0.03; visual mesh filename=../meshes/calf.stl scale=1 1 1
- link FR_foot: mass 0.05 -> 0.06
- link FR_hip: mass 2.15 -> 1.993; geometry collision cylinder length=0.04 radius=0.09; visual mesh filename=../meshes/hip.stl scale=1 1 1
- link FR_thigh: mass 4.3 -> 0.639; geometry collision box size=0.35 0.05 0.08; visual mesh filename=../meshes/thigh_mirror.stl scale=1 1 1
- link RL_calf: mass 1.05 -> 0.207; geometry collision box size=0.35 0.04 0.03; visual mesh filename=../meshes/calf.stl scale=1 1 1
- link RL_foot: mass 0.05 -> 0.06
- link RL_hip: mass 2.15 -> 1.993; geometry collision cylinder length=0.04 radius=0.09; visual mesh filename=../meshes/hip.stl scale=1 1 1
- link RL_thigh: mass 4.3 -> 0.639; geometry collision box size=0.35 0.05 0.08; visual mesh filename=../meshes/thigh.stl scale=1 1 1
- link RR_calf: mass 1.05 -> 0.207; geometry collision box size=0.35 0.04 0.03; visual mesh filename=../meshes/calf.stl scale=1 1 1
- link RR_foot: mass 0.05 -> 0.06
- link RR_hip: mass 2.15 -> 1.993; geometry collision cylinder length=0.04 radius=0.09; visual mesh filename=../meshes/hip.stl scale=1 1 1
- link RR_thigh: mass 4.3 -> 0.639; geometry collision box size=0.35 0.05 0.08; visual mesh filename=../meshes/thigh_mirror.stl scale=1 1 1
- link trunk: mass 29.45 -> 9.041; geometry collision box size=0.647 0.3 0.15; visual mesh filename=../meshes/trunk.stl scale=1 1 1
Joints:
- removed joint FL_calf_rotor_joint
- removed joint FL_hip_rotor_joint
- removed joint FL_thigh_rotor_joint
- removed joint FR_calf_rotor_joint
- removed joint FR_hip_rotor_joint
- removed joint FR_thigh_rotor_joint
- removed joint RL_calf_rotor_joint
- removed joint RL_hip_rotor_joint
- removed joint RL_thigh_rotor_joint
- removed joint RR_calf_rotor_joint
- removed joint RR_hip_rotor_joint
- removed joint RR_thigh_rotor_joint
- removed joint head_camera_1_joint
- removed joint head_camera_2_joint
- removed joint left_side_camera_joint
- removed joint right_side_camera_joint
- removed joint tail_camera_joint
- joint FL_calf_joint: limit lower=-2.6 upper=-0.6 effort=140 velocity=15.55 -> lower=-2.6 upper=-0.6 effort=100 velocity=20
- joint FL_hip_joint: limit lower=-0.75 upper=0.75 effort=91.0035 velocity=19.69 -> lower=-0.75 upper=0.75 effort=100 velocity=20
- joint FL_thigh_joint: limit lower=-1.0 upper=3.5 effort=93.33 velocity=23.32 -> lower=-1.0 upper=3.5 effort=100 velocity=20
- joint FR_calf_joint: limit lower=-2.6 upper=-0.6 effort=140 velocity=15.55 -> lower=-2.6 upper=-0.6 effort=100 velocity=20
- joint FR_hip_joint: limit lower=-0.75 upper=0.75 effort=91.0035 velocity=19.69 -> lower=-0.75 upper=0.75 effort=100 velocity=20
- joint FR_thigh_joint: limit lower=-1.0 upper=3.5 effort=93.33 velocity=23.32 -> lower=-1.0 upper=3.5 effort=100 velocity=20
- joint RL_calf_joint: limit lower=-2.6 upper=-0.6 effort=140 velocity=15.55 -> lower=-2.6 upper=-0.6 effort=100 velocity=20
- joint RL_hip_joint: limit lower=-0.75 upper=0.75 effort=91.0035 velocity=19.69 -> lower=-0.75 upper=0.75 effort=100 velocity=20
- joint RL_thigh_joint: limit lower=-1.0 upper=3.5 effort=93.33 velocity=23.32 -> lower=-1.0 upper=3.5 effort=100 velocity=20
- joint RR_calf_joint: limit lower=-2.6 upper=-0.6 effort=140 velocity=15.55 -> lower=-2.6 upper=-0.6 effort=100 velocity=20
- joint RR_hip_joint: limit lower=-0.75 upper=0.75 effort=91.0035 velocity=19.69 -> lower=-0.75 upper=0.75 effort=100 velocity=20
- joint RR_thigh_joint: limit lower=-1.0 upper=3.5 effort=93.33 velocity=23.32 -> lower=-1.0 upper=3.5 effort=100 velocity=20
